File: retroBuild/untitled.kicad_sch (KiCad schematic)
At the start: 134 parts, among them SW10 8*, SW11 9(, SW12 0), SW13 -_, SW14 =+, SW15 BSPC, SW16 PGUP, SW17 TAB, SW18 Q, SW19 W, SW2 `~, SW20 E, SW21 R, SW22 T, SW23 Y, SW24 U, SW25 I, SW26 O, SW27 P, SW28 [{, SW29 ]}, SW3 1!, SW30 \|, SW31 PGDN, SW32 CAPS, SW33 A, SW34 S, SW35 D, SW36 F, SW37 G, SW38 H, SW39 J, SW4 2@, SW40 K, SW41 L, SW42 ;:, SW43 '", SW45 ENTER, SW46 INSERT, SW47 LSHIFT, SW48 Z, SW49 X, SW5 3#, SW50 C, SW51 V, SW52 B, SW53 N, SW54 M, SW55 ,<, SW56 .>, SW57 /?, SW59 RSHIFT, SW6 4$, SW60 UP, SW61 DELETE, SW62 LCTRL, SW63 START, SW64 LALT, SW68 SPACE, SW7 5%, SW72 RALT, SW73 FUNC, SW74 LEFT, SW75 DOWN, SW76 RIGHT, SW8 6^, SW9 7&

Commit message: keys layed out in pcb view
Parts:
- D1, D10, D11, D12, D13, D14, D15, D16, D17, D18, D19, D2, D20, D21, D22, D23, D24, D25, D26, D27, D28, D29, D3, D30, D31, D32, D33, D34, D35, D36, D37, D38, D39, D4, D40, D41, D42, D44, D45, D46, D47, D48, D49, D5, D50, D51, D52, D53, D54, D55, D56, D58, D59, D6, D60, D61, D62, D63, D67, D7, D71, D72, D73, D74, D75, D8, D9: footprint (none) -> Diode_SMD:D_SOD-123
- SW10, SW11, SW12, SW13, SW14, SW16, SW18, SW19, SW2, SW20, SW21, SW22, SW23, SW24, SW25, SW26, SW27, SW28, SW29, SW3, SW31, SW33, SW34, SW35, SW36, SW37, SW38, SW39, SW4, SW40, SW41, SW42, SW43, SW46, SW48, SW49, SW5, SW50, SW51, SW52, SW53, SW54, SW55, SW56, SW57, SW6, SW60, SW61, SW7, SW74, SW75, SW76, SW8, SW9: footprint (none) -> Alps_MX_Stabilizers:MX-Alps-Hybrid-1U
- SW15: footprint (none) -> Alps_MX_Stabilizers:MX-Alps-Hybrid-2U
- SW17, SW30: footprint (none) -> Alps_MX_Stabilizers:MX-Alps-Hybrid-1.5U
- SW32, SW59: footprint (none) -> Alps_MX_Stabilizers:MX-Alps-Hybrid-1.75U
- SW45, SW47: footprint (none) -> Alps_MX_Stabilizers:MX-Alps-Hybrid-2.25U
- SW62, SW63, SW64, SW72, SW73: footprint (none) -> Alps_MX_Stabilizers:MX-Alps-Hybrid-1.25U
- SW68: footprint (none) -> Alps_MX_Stabilizers:MX-Alps-Hybrid-6.25U
